File: Hardware/THAT_1646_Breakout.brd (EAGLE design)
At the start: 48.3 x 20.3 mm, 20 parts, among them IC2 THAT1646, J2 OUTPUT, J6 CHASSIS

Commit message: Routed board.
Worked through initial checklist.
Parts:
- removed H5, H6, H7, H8: STAND-OFF, SparkFun-Electromechanical:STAND-OFF
- added FD1, FD2: FIDUCIALUFIDUCIAL, SparkFun-Aesthetics:MICRO-FIDUCIAL
- added LOGO1, LOGO2: SFE_LOGO_NAME.1_INCH, SparkFun-Aesthetics:SFE_LOGO_NAME_.1
- added LOGO3: SFE_LOGO_FLAME.2_INCH, SparkFun-Aesthetics:SFE_LOGO_FLAME_.2
- added LOGO4, LOGO5: OSHW-LOGOS, SparkFun-Aesthetics:OSHW-LOGO-S
- moved C7 10.2 mm to (22.9, 16.5), turned to 90 degrees
- moved C8 10.2 mm to (22.9, 3.81), turned to 270 degrees
- moved D1 4.75 mm to (17.3, 10.2), turned to 0 degrees
- moved L1 2.96 mm to (21.6, 13.0)
- moved IC2 2.84 mm to (8.89, 10.2)
- moved L2 2.84 mm to (21.6, 7.62)
- moved J2 2.54 mm to (45.7, 8.89)
- moved D2 2.18 mm to (13.5, 10.2), turned to 180 degrees
- moved C10 1.48 mm to (5.08, 3.05)
- moved JP2 1.27 mm to (21.0, 2.54)
- moved J6 1.27 mm to (44.5, 7.62)
- moved C9 1.08 mm to (8.13, 3.05)
- moved C12 0.92 mm to (15.7, 15.7)
- moved C11 0.92 mm to (15.7, 4.57)
Routing:
- net VCC: track 0.00 -> 30.9 mm, vias 0 -> 2
- net VNEG: track 0.00 -> 27.5 mm, vias 0 -> 2
- net N$9: track 0.00 -> 17.6 mm
- net N$8: track 0.00 -> 15.2 mm
- net N$11: track 0.00 -> 14.6 mm
- net N$10: track 0.00 -> 14.5 mm
- net N$16: track 0.00 -> 8.12 mm, vias 0 -> 1
- net N$14: track 0.00 -> 6.42 mm
- net N$13: track 0.00 -> 6.42 mm
- net GND-ISO: track 0.00 -> 1.14 mm, vias 0 -> 13
- net GND: track 0.00 -> 1.14 mm, vias 0 -> 15
Other:
- board size 48.3 x 20.3 mm -> 45.7 x 20.3 mm
- board text added: "All dimensions in inches"
- board text added: "Chassis"
- board text added: "Cut jumper to isolate chassis and circuit grounds"
- board text added: "Drill 3/8" hole to accomodate TRS jack"
- board text added: "THAT 1646 Breakout"
- board text added: "THAT 1646 OutSmarts Line Driver Breakout"

Commit message: Post-review updates.
Parts:
- removed C11, C12: 10uf, that-ics:PANASONIC_D
- removed C7, C8: 100pF, SparkFun-Capacitors:0603-CAP
- removed LOGO5: OSHW-LOGOS, SparkFun-Aesthetics:OSHW-LOGO-S
- added C3, C4: 10uf NP, that-ics:PANASONIC_D
- added C5, C6: 100pF, SparkFun-Capacitors:0603-CAP
- added FD3, FD4: FIDUCIALUFIDUCIAL, SparkFun-Aesthetics:MICRO-FIDUCIAL
- added J1: (no value), SparkFun-Connectors:1X04_NO_SILK_ALL_ROUND
- added J3: CHASSIS, SparkFun-Connectors:1X02_NO_SILK
- added J4: SN, SparkFun-Connectors:1X01_NO_SILK
- added LOGO6: SFE_LOGO_FLAME.2_INCH, SparkFun-Aesthetics:SFE_LOGO_FLAME_.2
- J5: value (none) -> TN; device SparkFun-Connectors:1X04_NO_SILK_ALL_ROUND -> SparkFun-Connectors:1X01_NO_SILK
- J6: value CHASSIS -> RN; device SparkFun-Connectors:1X02_NO_SILK -> SparkFun-Connectors:1X01_NO_SILK
- JP1: value JUMPER-PAD-2-NC_BY_TRACE -> GND-JOIN
- LOGO1, LOGO2: value SFE_LOGO_NAME.1_INCH -> OSHW-LOGOS; device SparkFun-Aesthetics:SFE_LOGO_NAME_.1 -> SparkFun-Aesthetics:OSHW-LOGO-S
- LOGO4: value OSHW-LOGOS -> SFE_LOGO_NAME.1_INCH; device SparkFun-Aesthetics:OSHW-LOGO-S -> SparkFun-Aesthetics:SFE_LOGO_NAME_.1
- moved LOGO2 33.8 mm to (7.37, 17.5)
- moved LOGO4 32.9 mm to (40.3, 16.5), flipped to the bottom
- moved J5 24.7 mm to (25.4, 1.27), turned to 0 degrees
- moved LOGO1 22.1 mm to (7.37, 17.5)
- moved J6 14.2 mm to (31.8, 1.27), turned to 0 degrees
- moved D1 3.81 mm to (13.5, 10.2), turned to 180 degrees
- moved D2 3.81 mm to (17.3, 10.2), turned to 0 degrees
- moved L2 2.90 mm to (20.8, 4.83)
- moved L1 1.70 mm to (20.8, 14.5)
- moved FD2 1.44 mm to (42.7, 0.76)
- moved FD1 1.27 mm to (1.02, 17.5)
- renumbered C10 to C2, C9 to C1, IC2 to IC1, JP2 to JP1
Connections:
- new net N$1: J2.RING-NORM, J6.1
- new net N$2: J2.TIP-NORM, J5.1
- new net N$3: J2.SLEEVE-NORM, J4.1
- net GND: now also J1.1; no longer J5.1
- net GND-ISO: now also C5.2, C6.2, J3.1, J3.2; no longer C7.2, C8.2, J6.1, J6.2
- net N$10: now also C3.-, D1.3; no longer C11.-, D2.3
- net N$11: now also C4.-, D2.3; no longer C12.-, D1.3
- net N$13: now also C4.+; no longer C12.+
- net N$14: now also C3.+; no longer C11.+
- net N$16: now also J1.4; no longer J5.4
- net N$8: now also C5.1; no longer C8.1
- net N$9: now also C6.1; no longer C7.1
- net VCC: now also J1.3; no longer J5.3
- net VNEG: now also J1.2; no longer J5.2
Routing:
- net N$2: track 0.00 -> 4.87 mm
- net N$1: track 0.00 -> 4.82 mm
- net N$3: track 0.00 -> 4.48 mm
- net VNEG: track 27.5 -> 26.0 mm
- net N$8: track 15.2 -> 16.7 mm
- net N$10: track 14.5 -> 13.1 mm
- net N$9: track 17.6 -> 16.9 mm
- net N$11: track 14.6 -> 15.2 mm
- net GND-ISO: vias 13 -> 15
Other:
- board text added: "Drill 0.440" (11mm) hole to accomodate TRS jack"
- board text added: "RN"
- board text added: "SN"
- board text added: "TN"
- board text removed: "Drill 3/8" hole to accomodate TRS jack"

Commit message: Updates from engineering checklist.
Parts:
- removed LOGO6: SFE_LOGO_FLAME.2_INCH, SparkFun-Aesthetics:SFE_LOGO_FLAME_.2
- added LOGO5: SFE_LOGO_NAME.1_INCH, SparkFun-Aesthetics:SFE_LOGO_NAME_.1
- D1, D2: value (none) -> BAV99
- J1: value (none) -> 1x4
- J2: value OUTPUT -> SN; device SparkFun-Connectors:AUDIO-JACK-.25-INCH-HORIZ-PTH -> SparkFun-Connectors:1X01_NO_SILK
- J4: value SN -> TN
- J5: value TN -> RN
- J6: value RN -> OUTPUT; device SparkFun-Connectors:1X01_NO_SILK -> SparkFun-Connectors:AUDIO-JACK-.25-INCH-HORIZ-PTH
- LOGO4: value SFE_LOGO_NAME.1_INCH -> SFE_LOGO_FLAME.2_INCH; device SparkFun-Aesthetics:SFE_LOGO_NAME_.1 -> SparkFun-Aesthetics:SFE_LOGO_FLAME_.2
- moved J4 19.1 mm to (25.4, 1.27)
- moved J6 15.9 mm to (45.7, 8.89), turned to 180 degrees
- moved LOGO4 10.7 mm to (34.8, 7.37), turned to 90 degrees
- moved J2 7.73 mm to (44.5, 1.27), turned to 0 degrees
- moved J5 6.35 mm to (31.8, 1.27)
- flipped FD1 to the bottom
- flipped FD2 to the bottom
- flipped FD3 to the top
- flipped FD4 to the top
Connections:
- net GND-ISO: now also J6.SLEEVE; no longer J2.SLEEVE
- net N$1: now also J5.1, J6.RING-NORM; no longer J2.RING-NORM, J6.1
- net N$2: now also J4.1, J6.TIP-NORM; no longer J2.TIP-NORM, J5.1
- net N$3: now also J2.1, J6.SLEEVE-NORM; no longer J2.SLEEVE-NORM, J4.1
- net N$8: now also J6.TIP; no longer J2.TIP
- net N$9: now also J6.RING; no longer J2.RING
Changed lines of the file:
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@@
 <setting verticaltext="up"/>
 </settings>
-<grid distance="0.05" unitdist="inch" unit="inch" style="lines" multiple="1" display="yes" altdistance="0.005" altunitdist="inch" altunit="inch"/>
+<grid distance="0.01" unitdist="inch" unit="inch" style="lines" multiple="1" display="yes" altdistance="0.005" altunitdist="inch" altunit="inch"/>
 <layers>
 <layer number="1" name="Top" color="4" fill="1" visible="yes" active="yes"/>
@@
 <layer number="37" name="tTest" color="7" fill="1" visible="no" active="yes"/>
 <layer number="38" name="bTest" color="7" fill="1" visible="no" active="yes"/>
-<layer number="39" name="tKeepout" color="4" fill="11" visible="no" active="yes"/>
-<layer number="40" name="bKeepout" color="1" fill="11" visible="no" active="yes"/>
+<layer number="39" name="tKeepout" color="4" fill="11" visible="yes" active="yes"/>
+<layer number="40" name="bKeepout" color="1" fill="11" visible="yes" active="yes"/>
 <layer number="41" name="tRestrict" color="4" fill="10" visible="no" active="yes"/>
 <layer number="42" name="bRestrict" color="1" fill="10" visible="no" active="yes"/>
@@
 <layer number="45" name="Holes" color="7" fill="1" visible="yes" active="yes"/>
 <layer number="46" name="Milling" color="3" fill="1" visible="no" active="yes"/>
-<layer number="47" name="Measures" color="7" fill="1" visible="no" active="yes"/>
+<layer number="47" name="Measures" color="7" fill="1" visible="yes" active="yes"/>
 <layer number="48" name="Document" color="7" fill="1" visible="no" active="yes"/>
 <layer number="49" name="Reference" color="7" fill="1" visible="no" active="yes"/>
@@
 <attribute name="PROD_ID" value="IC-13473" x="8.89" y="10.16" size="1.778" layer="27" rot="R180" display="off"/>
 </element>
-<element name="J2" library="SparkFun-Connectors" package="AUDIO-JACK-.25-INCH-HORIZ-PTH" value="OUTPUT" x="45.72" y="8.89" rot="R180">
+<element name="J6" library="SparkFun-Connectors" package="AUDIO-JACK-.25-INCH-HORIZ-PTH" value="OUTPUT" x="45.72" y="8.89" rot="R180">
 <attribute name="PROD_ID" value="CONN-12339" x="45.72" y="8.89" size="1.778" layer="27" rot="R180" display="off"/>
 <attribute name="SF_ID" value="COM-11144" x="45.72" y="8.89" size="1.778" layer="27" rot="R180" display="off"/>
@@
 <attribute name="PROD_ID" value="NDUC-12579" x="20.828" y="4.826" size="1.778" layer="27" display="off"/>
 </element>
-<element name="D2" library="SparkFun-DiscreteSemi" package="SOT23-3" value="" x="17.272" y="10.16">
+<element name="D2" library="SparkFun-DiscreteSemi" package="SOT23-3" value="BAV99" x="17.272" y="10.16">
 <attribute name="PROD_ID" value="DIO-10647" x="17.272" y="10.16" size="1.778" layer="27" font="vector" ratio="15" display="off"/>
 </element>
-<element name="D1" library="SparkFun-DiscreteSemi" package="SOT23-3" value="" x="13.462" y="10.16" rot="R180">
+<element name="D1" library="SparkFun-DiscreteSemi" package="SOT23-3" value="BAV99" x="13.462" y="10.16" rot="R180">
 <attribute name="PROD_ID" value="DIO-10647" x="13.462" y="10.16" size="1.778" layer="27" font="vector" ratio="15" rot="R180" display="off"/>
 </element>
@@
 <attribute name="PROD_ID" value="CAP-08604" x="5.08" y="3.048" size="1.778" layer="27" font="vector" ratio="15" rot="R90" display="off"/>
 </element>
-<element name="J1" library="SparkFun-Connectors" package="1X04_NO_SILK_ALL_ROUND" value="" x="1.27" y="6.35" rot="R90">
+<element name="J1" library="SparkFun-Connectors" package="1X04_NO_SILK_ALL_ROUND" value="1x4" x="1.27" y="6.35" rot="R90">
 <attribute name="PROD_ID" value="CONN-09696" x="1.27" y="6.35" size="1.778" layer="27" font="vector" ratio="15" rot="R90" display="off"/>
 </element>
 <element name="J3" library="SparkFun-Connectors" package="1X02_NO_SILK" value="CHASSIS" x="44.45" y="7.62" rot="R90"/>
-<element name="FD1" library="SparkFun-Aesthetics" package="MICRO-FIDUCIAL" value="FIDUCIALUFIDUCIAL" x="1.016" y="17.526"/>
-<element name="FD2" library="SparkFun-Aesthetics" package="MICRO-FIDUCIAL" value="FIDUCIALUFIDUCIAL" x="42.672" y="0.762"/>
-<element name="LOGO4" library="SparkFun-Aesthetics" package="SFE_LOGO_NAME_.1" value="SFE_LOGO_NAME.1_INCH" x="40.259" y="16.51" rot="MR0"/>
+<element name="FD3" library="SparkFun-Aesthetics" package="MICRO-FIDUCIAL" value="FIDUCIALUFIDUCIAL" x="1.016" y="17.526"/>
+<element name="FD4" library="SparkFun-Aesthetics" package="MICRO-FIDUCIAL" value="FIDUCIALUFIDUCIAL" x="42.672" y="0.762"/>
+<element name="LOGO5" library="SparkFun-Aesthetics" package="SFE_LOGO_NAME_.1" value="SFE_LOGO_NAME.1_INCH" x="40.259" y="16.51" rot="MR0"/>
 <element name="LOGO3" library="SparkFun-Aesthetics" package="SFE_LOGO_FLAME_.2" value="SFE_LOGO_FLAME.2_INCH" x="34.798" y="11.43" rot="R270"/>
 <element name="LOGO1" library="SparkFun-Aesthetics" package="OSHW-LOGO-S" value="OSHW-LOGOS" x="7.366" y="17.526"/>
 <element name="LOGO2" library="SparkFun-Aesthetics" package="OSHW-LOGO-S" value="OSHW-LOGOS" x="7.366" y="17.526" rot="MR0"/>
-<element name="J4" library="SparkFun-Connectors" package="1X01_NO_SILK" value="SN" x="44.45" y="1.27"/>
-<element name="J5" library="SparkFun-Connectors" package="1X01_NO_SILK" value="TN" x="25.4" y="1.27"/>
-<element name="J6" library="SparkFun-Connectors" package="1X01_NO_SILK" value="RN" x="31.75" y="1.27"/>
-<element name="LOGO6" library="SparkFun-Aesthetics" package="SFE_LOGO_FLAME_.2" value="SFE_LOGO_FLAME.2_INCH" x="34.798" y="7.366" rot="MR90"/>
-<element name="FD3" library="SparkFun-Aesthetics" package="MICRO-FIDUCIAL" value="FIDUCIALUFIDUCIAL" x="1.016" y="17.526" rot="MR0"/>
-<element name="FD4" library="SparkFun-Aesthetics" package="MICRO-FIDUCIAL" value="FIDUCIALUFIDUCIAL" x="42.672" y="0.762" rot="MR0"/>
+<element name="J2" library="SparkFun-Connectors" package="1X01_NO_SILK" value="SN" x="44.45" y="1.27"/>
+<element name="J4" library="SparkFun-Connectors" package="1X01_NO_SILK" value="TN" x="25.4" y="1.27"/>
+<element name="J5" library="SparkFun-Connectors" package="1X01_NO_SILK" value="RN" x="31.75" y="1.27"/>
+<element name="LOGO4" library="SparkFun-Aesthetics" package="SFE_LOGO_FLAME_.2" value="SFE_LOGO_FLAME.2_INCH" x="34.798" y="7.366" rot="MR90"/>
+<element name="FD1" library="SparkFun-Aesthetics" package="MICRO-FIDUCIAL" value="FIDUCIALUFIDUCIAL" x="1.016" y="17.526" rot="MR0"/>
+<element name="FD2" library="SparkFun-Aesthetics" package="MICRO-FIDUCIAL" value="FIDUCIALUFIDUCIAL" x="42.672" y="0.762" rot="MR0"/>
 <element name="C3" library="that-ics" package="PANASONIC_D" value="10uf NP" x="14.986" y="3.81" rot="R180">
 <attribute name="DK_PN" value="PCE4294TR-ND" x="14.986" y="3.81" size="1.778" layer="27" font="vector" ratio="15" rot="R180" display="off"/>
@@
 </signal>
 <signal name="GND-ISO">
-<contactref element="J2" pad="SLEEVE"/>
+<contactref element="J6" pad="SLEEVE"/>
 <contactref element="C5" pad="2"/>
 <contactref element="C6" pad="2"/>
@@
 <signal name="N$8">
 <contactref element="L2" pad="2"/>
-<contactref element="J2" pad="TIP"/>
+<contactref element="J6" pad="TIP"/>
 <contactref element="C5" pad="1"/>
 <wire x1="22.86" y1="6.096" x2="22.86" y2="4.826" width="0.254" layer="1"/>
@@
 </signal>
 <signal name="N$9">
-<contactref element="J2" pad="RING"/>
+<contactref element="J6" pad="RING"/>
 <contactref element="L1" pad="2"/>
 <contactref element="C6" pad="1"/>
@@
 <wire x1="10.9728" y1="12.954" x2="10.795" y2="12.7762" width="0.254" layer="1"/>
 <wire x1="17.272" y1="11.26" x2="17.272" y2="12.954" width="0.254" layer="1"/>
-<wire x1="18.454" y1="12.954" x2="19.978" y2="14.478" width="0.254" layer="1"/>
+<wire x1="18.454" y1="12.954" x2="18.879" y2="13.379" width="0.254" layer="1"/>
+<wire x1="18.879" y1="13.379" x2="19.978" y2="14.478" width="0.254" layer="1"/>
 <wire x1="17.272" y1="12.954" x2="18.454" y2="12.954" width="0.254" layer="1"/>
-<wire x1="17.386" y1="13.068" x2="17.272" y2="12.954" width="0.254" layer="1"/>
 <contactref element="C4" pad="-"/>
-<wire x1="17.386" y1="16.51" x2="17.386" y2="13.068" width="0.254" layer="1"/>
+<wire x1="17.386" y1="16.51" x2="17.386" y2="14.872" width="0.254" layer="1"/>
+<wire x1="17.386" y1="14.872" x2="18.879" y2="13.379" width="0.254" layer="1"/>
 </signal>
 <signal name="N$13">
@@
 </signal>
 <signal name="N$1">
-<contactref element="J2" pad="RING-NORM"/>
-<contactref element="J6" pad="1"/>
+<contactref element="J6" pad="RING-NORM"/>
+<contactref element="J5" pad="1"/>
 <wire x1="31.75" y1="1.27" x2="35.02" y2="4.54" width="0.254" layer="1"/>
 <wire x1="35.02" y1="4.54" x2="35.22" y2="4.54" width="0.254" layer="1"/>
 </signal>
 <signal name="N$2">
-<contactref element="J2" pad="TIP-NORM"/>
-<contactref element="J5" pad="1"/>
+<contactref element="J6" pad="TIP-NORM"/>
+<contactref element="J4" pad="1"/>
 <wire x1="25.4" y1="1.27" x2="28.67" y2="4.54" width="0.254" layer="1"/>
 <wire x1="28.67" y1="4.54" x2="28.92" y2="4.54" width="0.254" layer="1"/>
 </signal>
 <signal name="N$3">
-<contactref element="J2" pad="SLEEVE-NORM"/>
-<contactref element="J4" pad="1"/>
+<contactref element="J6" pad="SLEEVE-NORM"/>
+<contactref element="J2" pad="1"/>
 <wire x1="44.45" y1="1.27" x2="41.52" y2="4.2" width="0.254" layer="1"/>
 <wire x1="41.52" y1="4.2" x2="41.52" y2="4.54" width="0.254" layer="1"/>
